Commit message: фик пятой лабы

File: p5/ex05/robot3l/urdf/robot.xacro (robot description, xacro)
@@ -9,12 +9,11 @@
   <material name="gray"><color rgba="0.3 0.3 0.3 1"/></material>
   <!-- Base Link -->
-  <!-- Base Link -->
-  <link name="base_link">
-    <inertial>
-      <origin xyz="0 0 0" rpy="0 0 0"/>
-      <mass value="0.001"/>
-      <inertia ixx="1e-6" ixy="0" ixz="0" iyy="1e-6" iyz="0" izz="1e-6"/>
-    </inertial>
-  </link>
+  <link name="base_link"/>
+  <link name="base_footprint"/>
+  <joint name="base_footprint_joint" type="fixed">
+    <parent link="base_link"/>
+    <child link="base_footprint"/>
+    <origin rpy="0 0 0" xyz="0 0 -0.138"/>
+  </joint>
   <!-- Chassis -->
   <joint name="chassis_joint" type="fixed">
@@ -208,20 +207,89 @@
     </inertial>
   </link>
+    <!-- Lidar -->
+  <joint name="laser_joint" type="fixed">
+    <parent link="base_link"/>
+    <child link="laser_frame"/>
+    <origin xyz="0.1 0 0.212" rpy="0 0 0"/>
+  </joint>
+  <link name="laser_frame">
+    <visual>
+      <geometry>
+        <cylinder radius="0.05" length="0.04"/>
+      </geometry>
+      <material name="black"/>
+    </visual>
+    <visual>
+      <origin xyz="0 0 -0.05"/>
+      <geometry>
+        <cylinder radius="0.01" length="0.1"/>
+      </geometry>
+      <material name="black"/>
+    </visual>
+    <collision>
+      <geometry>
+        <cylinder radius="0.05" length="0.04"/>
+      </geometry>
+    </collision>
+    <inertial>
+      <origin xyz="0 0 0" rpy="0 0 0"/>
+      <mass value="0.1" />
+      <inertia ixx="${(1/12) * 0.1 * (3*0.05*0.05 + 0.04*0.04)}" ixy="0.0" ixz="0.0"
+               iyy="${(1/12) * 0.1 * (3*0.05*0.05 + 0.04*0.04)}" iyz="0.0"
+               izz="${(1/2) * 0.1 * (0.05*0.05)}" />
+    </inertial>
+  </link>
+  <gazebo reference="laser_frame">
+    <material>Gazebo/Black</material>
+    <sensor name='laser_sensor_frame' type='gpu_lidar'>
+        <gz_frame_id>laser_frame</gz_frame_id>
+        <pose>0 0 0 0 0 0</pose>
+        <visualize>true</visualize>
+        <always_on>true</always_on>
+        <update_rate>20</update_rate>
+        <ray>
+            <scan>
+                <horizontal>
+                    <samples>360</samples>
+                    <min_angle>-3.14</min_angle>
+                    <max_angle>3.14</max_angle>
+                </horizontal>
+            </scan>
+            <range>
+                <min>0.3</min>
+                <max>12</max>
+            </range>
+            <noise>
+                <type>gaussian</type>
+                <mean>0.0</mean>
+                <stddev>0.007</stddev>
+            </noise>
+        </ray>
+    </sensor>
+  </gazebo>
   <!-- Plugins -->
-    <gazebo>
-    <!-- Публикуем состояние джойнтов в /joint_states -->
-    <plugin filename="gz-sim-joint-state-publisher-system" name="gz::sim::systems::JointStatePublisher">
+<gazebo>
+    <plugin filename="libgz-sim-joint-state-publisher-system.so" name="gz::sim::systems::JointStatePublisher"/>
+    <plugin filename="libgz-sim-diff-drive-system.so" name="gz::sim::systems::DiffDrive">
+      <left_joint>left_wheel_joint</left_joint>
+      <right_joint>right_wheel_joint</right_joint>
+      <child_frame_id>robot/base_link</child_frame_id>
+      <wheel_separation>0.291</wheel_separation>
+      <wheel_radius>0.1</wheel_radius>
+        <odom_update_frequency>50</odom_update_frequency>
+    <!-- ВАЖНО! Новые параметры TF в Sim8 -->
+    <odom_frame>odom</odom_frame>                 <!-- новое имя -->
+    <base_frame>base_link</base_frame>            <!-- новое имя -->
+    <publish_tf>true</publish_tf>                 <!-- работает -->
+    <!-- ЭТО КРИТИЧЕСКОЕ ЗНАЧЕНИЕ ДЛЯ Sim8 -->
+    <publish_odom>true</publish_odom>             <!-- включает одометрию -->
+    <publish_cmd>true</publish_cmd>               <!-- включает cmd_vel -->
     </plugin>
-    <!-- DiffDrive для управления колесами -->
-    <plugin filename="gz-sim-diff-drive-system" name="gz::sim::systems::DiffDrive">
-    <left_joint>left_wheel_joint</left_joint>
-    <right_joint>right_wheel_joint</right_joint>
-    <wheel_separation>0.291</wheel_separation>
-    <wheel_radius>0.25</wheel_radius>
+  </gazebo>
+  <gazebo>
+    <plugin filename="gz-sim-sensors-system"
+                    name="gz::sim::systems::Sensors">
+                <render_engine>ogre2</render_engine>
     </plugin>
-    <plugin filename="gz-sim-odometry-publisher-system" name="gz::sim::systems::OdometryPublisher">
-    <topic>odometry</topic>
-    <odom_frame>odom</odom_frame>
-    <robot_base_frame>base_link</robot_base_frame>
-    </plugin>
-  </gazebo>
+  </gazebo>
+</robot>
